Commit message: add transform publisher

File: ros_ws/src/morbo_bringup/urdf/morbo.urdf (robot description, URDF)
Before this commit: robot morbo, 6 links, 5 joints
Joints:
- joint wheel_back_left_joint: type continuous -> fixed
- joint wheel_back_right_joint: type continuous -> fixed
- joint wheel_front_left_joint: type continuous -> fixed
- joint wheel_front_right_joint: type continuous -> fixed

Commit message: add laser frame

File: ros_ws/src/morbo_bringup/urdf/morbo.urdf (robot description, URDF)
Before this commit: robot morbo, 6 links, 5 joints
Links:
- added link laser; visual cylinder length=0.055 radius=0.05
Joints:
- added joint lidar_joint: type fixed, parent base_link, child laser, origin xyz=0.11 0 0.10 rpy=0 0 -3.14

Commit message: add nav bringup script

File: ros_ws/src/morbo_bringup/urdf/morbo.urdf (robot description, URDF)
Before this commit: robot morbo, 7 links, 6 joints
Links:
- removed link laser
- added link base_scan; visual cylinder length=0.055 radius=0.05
Joints:
- joint lidar_joint: child laser -> base_scan
